Commit message: d6

File: module06/ex05/my_robot/robot_description/urdf/gazebo.urdf.xacro (robot description, xacro)
@@ -35,4 +35,7 @@
                 <render_engine>ogre2</render_engine>
         </plugin>
+        <plugin filename="gz-sim-imu-system"
+            name="gz::sim::systems::Imu">
+        </plugin>
     </gazebo>
 </robot>

File: module06/ex05/my_robot/robot_description/urdf/robot.urdf.xacro (robot description, xacro)
@@ -3,5 +3,5 @@
     <xacro:include filename="$(find robot_description)/urdf/gazebo.urdf.xacro" />
     <xacro:include filename="$(find robot_description)/urdf/lidar.urdf.xacro" />
-    <!-- <xacro:include filename="$(find robot_description)/urdf/depth.urdf.xacro" /> -->
+    <xacro:include filename="$(find robot_description)/urdf/depth.urdf.xacro" />
     <xacro:property name="chassis_length" value="0.335"/>
     <xacro:property name="chassis_width" value="0.265"/>
@@ -161,5 +161,5 @@
     </gazebo>
      <!-- IMU SENSOR -->
-    <!-- <joint name="imu_sensor_joint" type="fixed">
+    <joint name="imu_sensor_joint" type="fixed">
         <origin xyz="0.11 0.0 0.07" rpy="0 0 0"/>
         <parent link="base_link"/>
@@ -197,5 +197,5 @@
             <pose>0 0 0 0 0 0</pose>
         </sensor>
-    </gazebo> -->
+    </gazebo>
     <!-- END IMU SENSOR -->
 </robot>
